File: ControlUnit/ButtonLEDsController/ButtonLEDsController.kicad_pcb (KiCad board)
At the start: 2 copper layers, 100.1 x 90.1 mm, 39 parts, among them U1 NodeMCU1.0(ESP-12E)

Commit message: 1mm thickness for all tacks
Other:
- net class Default: trace_width 0.25 -> 1

Commit message: prepared to order pcbs
Parts:
- D13: value DisplayBacklight -> LED
- D14, D15: value (none) -> LED_ARGB; footprint LEDs:LED_D5.0mm-4 -> Pin_Headers:Pin_Header_Straight_1x04
- J1: value (none) -> Conn_02x15_Odd_Even
- J2: value (none) -> Conn_01x03
- J3, J4, J5: value (none) -> Conn_01x01
- J6: value (none) -> Conn_01x02_Female
- Q1: value (none) -> IRLZ34N
- Q2: value (none) -> Q_PNP_EBC
- Q3, Q4, Q5, Q6, Q7, Q8: value (none) -> Q_NPN_EBC
- R1: value 10k -> 10kR
- moved D15 2.06 mm to (82.6, 53.2), turned to 0 degrees
- moved D14 1.27 mm to (82.4, 23.6), turned to 0 degrees
Connections:
- J1 pad 3: (no net) -> Net-(J1-Pad3)
- J1 pad 5: (no net) -> Net-(J1-Pad5)
- U1 pad 2: (no net) -> Net-(U1-Pad2)
- U1 pad 3: (no net) -> Net-(U1-Pad3)
Routing:
- net +5V: track 173.6 -> 161.1 mm
- net Net-(Q7-Pad2): track 5.73 -> 10.9 mm
- net Net-(D14-Pad4): track 12.8 -> 11.8 mm
- net Net-(D15-Pad3): track 10.9 -> 11.5 mm
- net Net-(D14-Pad3): track 11.0 -> 11.6 mm
Other:
- board size 100.1 x 90.1 mm -> 94 x 90 mm
