File: ControlUnit/ButtonLEDsController/ButtonLEDsController.sch (KiCad schematic (older format))
At the start: 39 parts, among them J1 Conn_02x15_Odd_Even, J2 Conn_01x03, J3 Conn_01x01, J4 Conn_01x01, J5 Conn_01x01, J6 Conn_01x02_Female, Q1 IRLZ34N, Q2 Q_PNP_EBC, Q3 Q_NPN_EBC, Q4 Q_NPN_EBC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

Commit message: prepared to order pcbs
Parts:
- D14, D15: footprint LEDs:LED_D5.0mm-4 -> Pin_Headers:Pin_Header_Straight_1x04
Changed lines of the file:
@@
 F 0 "D14" H 13250 3270 50  0000 C CNN
 F 1 "LED_ARGB" H 13250 2550 50  0000 C CNN
-F 2 "LEDs:LED_D5.0mm-4" H 13250 2850 50  0001 C CNN
+F 2 "Pin_Headers:Pin_Header_Straight_1x04" H 13250 2850 50  0001 C CNN
 F 3 "" H 13250 2850 50  0001 C CNN
 	1    13250 2900
@@
 F 0 "D15" H 13250 5420 50  0000 C CNN
 F 1 "LED_ARGB" H 13250 4700 50  0000 C CNN
-F 2 "LEDs:LED_D5.0mm-4" H 13250 5000 50  0001 C CNN
+F 2 "Pin_Headers:Pin_Header_Straight_1x04" H 13250 5000 50  0001 C CNN
 F 3 "" H 13250 5000 50  0001 C CNN
 	1    13250 5050
